Commit message: Prefix with twizy_ instead of sample_
Following this Autoware guide: https://autowarefoundation.github.io/autoware-documentation/main/how-to-guides/integrating-autoware/creating-vehicle-and-sensor-model/creating-vehicle-model/#creating-a-vehicle-model-for-autoware

File: twizy_vehicle_description/urdf/vehicle.xacro (robot description, xacro)
@@ -2,5 +2,5 @@
 <robot xmlns:xacro="http://ros.org/wiki/xacro">
   <!-- load parameter -->
-  <xacro:property name="vehicle_info" value="${xacro.load_yaml('$(find sample_vehicle_description)/config/vehicle_info.param.yaml')}"/>
+  <xacro:property name="vehicle_info" value="${xacro.load_yaml('$(find twizy_vehicle_description)/config/vehicle_info.param.yaml')}"/>
   <!-- vehicle body -->
   <link name="base_link">
@@ -8,5 +8,5 @@
       <origin xyz="${vehicle_info['/**']['ros__parameters']['wheel_base']/2.0} 0 0" rpy="${pi/2.0} 0 ${pi}"/>
       <geometry>
-        <mesh filename="package://sample_vehicle_description/mesh/lexus.dae" scale="1 1 1"/>
+        <mesh filename="package://twizy_vehicle_description/mesh/lexus.dae" scale="1 1 1"/>
       </geometry>
     </visual>

Commit message: Add urdf and update vehicle interface launch

File: twizy_vehicle_description/urdf/vehicle.xacro (robot description, xacro)
@@ -1,14 +1,49 @@
 <?xml version="1.0"?>
-<robot xmlns:xacro="http://ros.org/wiki/xacro">
-  <!-- load parameter -->
-  <xacro:property name="vehicle_info" value="${xacro.load_yaml('$(find twizy_vehicle_description)/config/vehicle_info.param.yaml')}"/>
-  <!-- vehicle body -->
-  <link name="base_link">
-    <visual>
-      <origin xyz="${vehicle_info['/**']['ros__parameters']['wheel_base']/2.0} 0 0" rpy="${pi/2.0} 0 ${pi}"/>
-      <geometry>
-        <mesh filename="package://twizy_vehicle_description/mesh/lexus.dae" scale="1 1 1"/>
-      </geometry>
-    </visual>
-  </link>
+<!--
+Copyright (c) 2020 StreetDrone Limited
+Author:  Efimia Panagiotaki
+All rights reserved
+-->
+<robot name="sd_twizy" xmlns:xacro="http://www.ros.org/wiki/xacro">
+  <xacro:include filename="$(find twizy_vehicle_description)/urdf/bases/sd_twizy_body.gazebo.xacro" />
+  <xacro:macro name="sd_twizy_base" params="name">
+    <xacro:property name="depth" value="2.352"/>
+    <xacro:property name="height" value="1.7"/>
+    <xacro:property name="width" value="1.431"/>
+    <xacro:property name="base_mass" value="435"/>
+    <xacro:property name="clearance" value="0.281"/>
+    <xacro:property name = "wheelbase" value="1.686"/>
+    <link name="base_link">
+      <visual>
+        <origin xyz="0 0 0" rpy="0 0 0" />
+        <geometry>
+          <box size="0.001 0.001 0.001" />
+        </geometry>
+      </visual>
+    </link>
+    <joint name="chassis_joint" type="fixed">
+      <origin xyz="${wheelbase / 2} 0 0" rpy="0 0 0"/>
+      <parent link="base_link"/>
+      <child link="chassis"/>
+    </joint>
+    <link name="chassis">
+      <inertial>
+        <mass value="${base_mass}"/>
+        <origin xyz="0 0 0"/>
+        <inertia ixx="243.175" ixy="0" ixz="0" iyy="430.166" iyz="0" izz="430.166"/>
+      </inertial>
+      <visual>
+        <origin xyz="0 0 0" rpy="0 0 1.57079632679"/>
+        <geometry>
+          <mesh filename="file://$(find twizy_vehicle_description)/meshes/SDTwizy.stl" scale="0.01 0.01 0.01"/>
+        </geometry>
+      </visual>
+      <collision>
+        <origin xyz="0 0 0" rpy="0 0 1.57079632679"/>
+        <geometry>
+          <mesh filename="file://$(find twizy_vehicle_description)/meshes/SDTwizy_collision.stl" scale="0.01 0.01 0.01"/>
+        </geometry>
+      </collision>
+    </link>
+  </xacro:macro>
 </robot>

Commit message: Add correct urdf/xacro from SD
https://github.com/streetdrone-home/SD-TwizyModel/tree/master/streetdrone_model/sd_description

File: twizy_vehicle_description/urdf/vehicle.xacro (robot description, xacro)
@@ -6,44 +6,84 @@
 -->
 <robot name="sd_twizy" xmlns:xacro="http://www.ros.org/wiki/xacro">
-  <xacro:include filename="$(find twizy_vehicle_description)/urdf/bases/sd_twizy_body.gazebo.xacro" />
-  <xacro:macro name="sd_twizy_base" params="name">
-    <xacro:property name="depth" value="2.352"/>
-    <xacro:property name="height" value="1.7"/>
-    <xacro:property name="width" value="1.431"/>
-    <xacro:property name="base_mass" value="435"/>
-    <xacro:property name="clearance" value="0.281"/>
-    <xacro:property name = "wheelbase" value="1.686"/>
-    <link name="base_link">
-      <visual>
-        <origin xyz="0 0 0" rpy="0 0 0" />
-        <geometry>
-          <box size="0.001 0.001 0.001" />
-        </geometry>
-      </visual>
-    </link>
-    <joint name="chassis_joint" type="fixed">
-      <origin xyz="${wheelbase / 2} 0 0" rpy="0 0 0"/>
-      <parent link="base_link"/>
-      <child link="chassis"/>
-    </joint>
-    <link name="chassis">
-      <inertial>
-        <mass value="${base_mass}"/>
-        <origin xyz="0 0 0"/>
-        <inertia ixx="243.175" ixy="0" ixz="0" iyy="430.166" iyz="0" izz="430.166"/>
-      </inertial>
-      <visual>
-        <origin xyz="0 0 0" rpy="0 0 1.57079632679"/>
-        <geometry>
-          <mesh filename="file://$(find twizy_vehicle_description)/meshes/SDTwizy.stl" scale="0.01 0.01 0.01"/>
-        </geometry>
-      </visual>
-      <collision>
-        <origin xyz="0 0 0" rpy="0 0 1.57079632679"/>
-        <geometry>
-          <mesh filename="file://$(find twizy_vehicle_description)/meshes/SDTwizy_collision.stl" scale="0.01 0.01 0.01"/>
-        </geometry>
-      </collision>
-    </link>
-  </xacro:macro>
+  <!-- ***************** -->
+  <!-- Imported elements -->
+  <!-- ***************** -->
+  <xacro:include filename="$(find twizy_vehicle_description)/urdf/bases/sd_twizy_body.urdf.xacro" />
+  <xacro:include filename="$(find twizy_vehicle_description)/urdf/wheels/sd_twizy_suspension.urdf.xacro" />
+  <xacro:include filename="$(find twizy_vehicle_description)/urdf/sensors/VLP-16.urdf.xacro"/>
+  <xacro:include filename="$(find twizy_vehicle_description)/urdf/sensors/cameras.urdf.xacro"/>
+  <!-- *************** -->
+  <!-- Robots Elements -->
+  <!-- *************** -->
+  <xacro:sd_twizy_base name="sd_twizy"/>
+  <xacro:RL_wheel/>
+  <xacro:RR_wheel/>
+  <xacro:FL_wheel/>
+  <xacro:FR_wheel/>
+  <!-- Sensors -->
+  <xacro:VLP-16  parent="chassis" name="velodyne" topic="/points_raw" hz="10" samples="1875">
+    <origin xyz="-0.681 0 1.445" rpy="0 -${1.5*M_PI/180.0} 0"/>
+  </xacro:VLP-16>
+  <xacro:blackfly_camera frlr_prefix="front" lrc_prefix="left">
+    <origin xyz="-0.04 0.12 1.3" rpy="0 0.087 0"/>
+  </xacro:blackfly_camera>
+  <xacro:blackfly_camera frlr_prefix="front" lrc_prefix="right">
+    <origin xyz="-0.04 -0.12 1.3" rpy="0 0.087 0"/>
+  </xacro:blackfly_camera>
+  <xacro:blackfly_camera frlr_prefix="front" lrc_prefix="center">
+    <origin xyz="-0.04 0 1.3" rpy="0 0.087 0"/>
+  </xacro:blackfly_camera>
+  <xacro:blackfly_camera frlr_prefix="rear" lrc_prefix="center">
+    <origin xyz="-1.26 0 1.28" rpy="0 0.2618 3.14"/>
+  </xacro:blackfly_camera>
+  <xacro:blackfly_camera frlr_prefix="right" lrc_prefix="forward">
+    <origin xyz="-0.95 -0.42 1.2" rpy="0 0.244 -1.12"/>
+  </xacro:blackfly_camera>
+  <xacro:blackfly_camera frlr_prefix="right" lrc_prefix="rearward">
+    <origin xyz="-1.05 -0.42 1.2" rpy="0 0.244 -2.18"/>
+  </xacro:blackfly_camera>
+  <xacro:blackfly_camera frlr_prefix="left" lrc_prefix="forward">
+    <origin xyz="-0.95 0.4 1.2" rpy="0 0.2967 1.12"/>
+  </xacro:blackfly_camera>
+  <xacro:blackfly_camera frlr_prefix="left" lrc_prefix="rearward">
+    <origin xyz="-1.05 0.39 1.2" rpy="0 0.2967 2.18"/>
+  </xacro:blackfly_camera>
+  <gazebo>
+    <plugin name="sd_control" filename="libSdControlPlugin.so">
+      <chassis>base_link</chassis>
+      <front_left_wheel>front_left_wheel_joint</front_left_wheel>
+      <front_right_wheel>front_right_wheel_joint</front_right_wheel>
+      <front_left_wheel_steering>front_left_steer_joint</front_left_wheel_steering>
+      <front_right_wheel_steering>front_right_steer_joint</front_right_wheel_steering>
+      <back_left_wheel>rear_left_wheel_joint</back_left_wheel>
+      <back_right_wheel>rear_right_wheel_joint</back_right_wheel>
+      <fl_wheel_steering_p_gain>1e4</fl_wheel_steering_p_gain>
+      <fr_wheel_steering_p_gain>1e4</fr_wheel_steering_p_gain>
+      <fl_wheel_steering_i_gain>0</fl_wheel_steering_i_gain>
+      <fr_wheel_steering_i_gain>0</fr_wheel_steering_i_gain>
+      <fl_wheel_steering_d_gain>3e2</fl_wheel_steering_d_gain>
+      <fr_wheel_steering_d_gain>3e2</fr_wheel_steering_d_gain>
+      <max_speed>22</max_speed>
+      <max_torque>250</max_torque>
+      <front_brake_torque>260</front_brake_torque>
+      <back_brake_torque>260</back_brake_torque>
+      <chassis_aero_force_gain>0.63045</chassis_aero_force_gain>
+    </plugin>
+  </gazebo>
+  <gazebo>
+    <plugin name="p3d" filename="libgazebo_ros_p3d.so">
+      <bodyName>base_link</bodyName>
+      <topicName>base_pose_ground_truth</topicName>
+      <frameName>map</frameName>
+      <updateRate>100.0</updateRate>
+    </plugin>
+  </gazebo>
+  <gazebo>
+    <plugin name="joint_state_publisher" filename="libgazebo_ros_joint_state_publisher.so">
+      <robotNamespace>/sd_twizy</robotNamespace>
+      <jointName>front_left_wheel_joint, front_right_wheel_joint, front_left_steer_joint, front_right_steer_joint, rear_left_wheel_joint, rear_right_wheel_joint</jointName>
+      <updateRate>100.0</updateRate>
+      <alwaysOn>true</alwaysOn>
+    </plugin>
+  </gazebo>
 </robot>
