Commit message: Comment out materials causing warnings

File: twizy_vehicle_description/urdf/sensors/cameras.urdf.xacro (robot description, xacro)
@@ -26,5 +26,5 @@
           <box size="0.026 0.026 0.0203"/>
         </geometry>
-        <material name="red"/>
+        <!-- <material name="red"/> -->
       </visual>
       <inertial>

File: twizy_vehicle_description/urdf/wheels/sd_twizy_suspension.urdf.xacro (robot description, xacro)
@@ -77,5 +77,5 @@
         <cylinder radius="${front_tyre_radius}" length="${front_tyre_width}"/>
       </geometry>
-      <material name="tire_mat"/>
+      <!-- <material name="tire_mat"/> -->
     </visual>
   </link>
@@ -97,5 +97,5 @@
         <cylinder radius="${front_tyre_radius}" length="${front_tyre_width}"/>
       </geometry>
-      <material name="tire_mat"/>
+      <!-- <material name="tire_mat"/> -->
     </visual>
   </link>
@@ -117,5 +117,5 @@
         <cylinder radius="${rear_tyre_radius}" length="${rear_tyre_width}"/>
       </geometry>
-      <material name="tire_mat"/>
+      <!-- <material name="tire_mat"/> -->
     </visual>
   </link>
@@ -137,5 +137,5 @@
         <cylinder radius="${rear_tyre_radius}" length="${rear_tyre_width}"/>
       </geometry>
-      <material name="tire_mat"/>
+      <!-- <material name="tire_mat"/> -->
     </visual>
   </link>
